File: rp2040-launchpad-PCB.kicad_pcb (KiCad board)
At the start: 2 copper layers, 58.4 x 83.8 mm, 127 parts, among them J1 Target Isolation Jumpers, J10 PWR Header, J11 LP Extension Heder, J12 LP Header right, J13 PWR Header, J2 Jumper, J3 LiPo 3,7V Batt., J4 Jumper, J5 DBG_PRGM, J6 UART_DBG, J7 DGB Exp. Header, J8 Jumper, J9 LP Header left, SW1 Switch_SP3T, SW2 RESET, SW3 BOOT, U1 MCP73831, U10 WS2812B-2020, U11 WS2812B-2020, U12 WS2812B-2020, U13 WS2812B-2020, U14 WS2812B-2020, U15 WS2812B-2020, U16 WS2812B-2020, U2 XC9142B50C, U3 XC6220B33, U4 25Q32, U5 RP2040, U6 25Q64, U7 APS6404L-3SQR, U8 RP2350_80QFN, U9 WS2812B-2020, Y1 12MHz, Y2 12MHz

Commit message: small change to PCB (GND area under MCU).
Routing:
- net GND: vias 96 -> 98
Changed lines of the file:
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@@
+	)
+	(via
+		(at 143.129 114.935)
+		(size 0.8)
+		(drill 0.4)
+		(layers "F.Cu" "B.Cu")
+		(net 2)
 	)
 	(via
@@
 		(size 0.8)
 		(drill 0.4)
+		(layers "F.Cu" "B.Cu")
+		(net 2)
+	)
+	(via
+		(at 143.129 119.634)
+		(size 0.8)
+		(drill 0.4)
