File: rp2350b-launchpad-PCB.kicad_pcb (KiCad board)
At the start: 2 copper layers, 58.4 x 83.8 mm, 127 parts, among them J1 Target Isolation Jumpers, J10 PWR Header, J11 LP Extension Heder, J12 LP Header right, J13 PWR Header, J2 Jumper, J3 LiPo 3,7V Batt., J4 Jumper, J5 DBG_PRGM, J6 UART_DBG, J7 DGB Exp. Header, J8 Jumper, J9 LP Header left, SW1 Switch_SP3T, SW2 RESET, SW3 BOOT, U1 MCP73831, U10 WS2812B-2020, U11 WS2812B-2020, U12 WS2812B-2020, U13 WS2812B-2020, U14 WS2812B-2020, U15 WS2812B-2020, U16 WS2812B-2020, U2 XC9142B50C, U3 XC6220B33, U4 25Q32, U5 RP2040, U6 25Q64, U7 APS6404L-3SQR, U8 RP2350_80QFN, U9 WS2812B-2020, Y1 12MHz, Y2 12MHz

Commit message: Renamed files.
Parts:
- G*** (x2): footprint rp2040-launchpad-PCB:Lauchpad-Energia-Logo -> rp2350b-launchpad-PCB:Lauchpad-Energia-Logo
- G***: footprint rp2040-launchpad-PCB:Lauchpad-Logo -> rp2350b-launchpad-PCB:Lauchpad-Logo
- G*** (x2): footprint rp2040-launchpad-PCB:raspberry -> rp2350b-launchpad-PCB:raspberry
Changed lines of the file:
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@@
 		(property ki_fp_filters "Connector*:*_2x??_*")
 		(sheetname "Stammblatt")
-		(sheetfile "rp2040-launchpad-PCB.kicad_sch")
+		(sheetfile "rp2350b-launchpad-PCB.kicad_sch")
 		(attr through_hole)
 		(fp_line
@@
 		)
 	)
-	(footprint "rp2040-launchpad-PCB:Lauchpad-Energia-Logo"
+	(footprint "rp2350b-launchpad-PCB:Lauchpad-Energia-Logo"
 		(layer "F.Cu")
 		(at 146.653035 139.382203)
@@
 		)
 	)
-	(footprint "rp2040-launchpad-PCB:Lauchpad-Logo"
+	(footprint "rp2350b-launchpad-PCB:Lauchpad-Logo"
 		(layer "F.Cu")
 		(at 151.384 82.804)
@@
 		)
 	)
-	(footprint "rp2040-launchpad-PCB:raspberry"
+	(footprint "rp2350b-launchpad-PCB:raspberry"
 		(layer "F.Cu")
 		(at 152.4 101.6)
@@
 		)
 	)
-	(footprint "rp2040-launchpad-PCB:Lauchpad-Energia-Logo"
+	(footprint "rp2350b-launchpad-PCB:Lauchpad-Energia-Logo"
 		(layer "B.Cu")
 		(at 138.080966 133.286203 180)
@@
 		)
 	)
-	(footprint "rp2040-launchpad-PCB:raspberry"
+	(footprint "rp2350b-launchpad-PCB:raspberry"
 		(layer "B.Cu")
 		(at 132.715 109.347 180)

Commit message: Fixes to manual renaming...
Parts:
- J3: footprint rp2350-launchpad:JST-S2B-PH-KL -> rp2350b-launchpad-PCB:JST-S2B-PH-KL
- S1, S2, SW2: footprint rp2350-launchpad:DIPT-1188E -> rp2350b-launchpad-PCB:DIPT-1188E
- SW1: footprint rp2350-launchpad:PCM13SMTR -> rp2350b-launchpad-PCB:PCM13SMTR
- SW3: footprint rp2350-launchpad:KMR2-Switch -> rp2350b-launchpad-PCB:KMR2-Switch
- U10, U11, U12, U13, U14, U15, U16, U9: footprint rp2350-launchpad:WS2812B-2020 -> rp2350b-launchpad-PCB:WS2812B-2020
- U5: footprint rp2350-launchpad:QFN40P700X700X90-57N -> rp2350b-launchpad-PCB:QFN40P700X700X90-57N
- USB1, USB2: footprint rp2350-launchpad:USB-C-GCT-USB4105 -> rp2350b-launchpad-PCB:USB-C-GCT-USB4105
Changed lines of the file:
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@@
 		)
 	)
-	(footprint "rp2350-launchpad:DIPT-1188E"
+	(footprint "rp2350b-launchpad-PCB:DIPT-1188E"
 		(layer "F.Cu")
 		(at 132.722 148.494)
@@
 			)
 		)
-		(property "Footprint" "rp2350-launchpad:DIPT-1188E"
+		(property "Footprint" "rp2350b-launchpad-PCB:DIPT-1188E"
 			(at 0 0 0)
 			(layer "F.Fab")
@@
 		)
 	)
-	(footprint "rp2350-launchpad:QFN40P700X700X90-57N"
+	(footprint "rp2350b-launchpad-PCB:QFN40P700X700X90-57N"
 		(layer "F.Cu")
 		(at 151.638 82.55)
@@
 			)
 		)
-		(property "Footprint" "rp2350-launchpad:QFN40P700X700X90-57N"
+		(property "Footprint" "rp2350b-launchpad-PCB:QFN40P700X700X90-57N"
 			(at 0 0 0)
 			(layer "F.Fab")
@@
 		)
 	)
-	(footprint "rp2350-launchpad:WS2812B-2020"
+	(footprint "rp2350b-launchpad-PCB:WS2812B-2020"
 		(layer "F.Cu")
 		(at 142.24 139.446 90)
@@
 			)
 		)
-		(property "Footprint" "rp2350-launchpad:WS2812B-2020"
+		(property "Footprint" "rp2350b-launchpad-PCB:WS2812B-2020"
 			(at 0 0 90)
 			(layer "F.Fab")
@@
 		)
 	)
-	(footprint "rp2350-launchpad:WS2812B-2020"
+	(footprint "rp2350b-launchpad-PCB:WS2812B-2020"
 		(layer "F.Cu")
 		(at 144.78 139.446 90)
@@
 			)
 		)
-		(property "Footprint" "rp2350-launchpad:WS2812B-2020"
+		(property "Footprint" "rp2350b-launchpad-PCB:WS2812B-2020"
 			(at 0 0 90)
 			(layer "F.Fab")
@@
 		)
 	)
-	(footprint "rp2350-launchpad:WS2812B-2020"
+	(footprint "rp2350b-launchpad-PCB:WS2812B-2020"
 		(layer "F.Cu")
 		(at 147.32 139.446 90)
@@
 			)
 		)
-		(property "Footprint" "rp2350-launchpad:WS2812B-2020"
+		(property "Footprint" "rp2350b-launchpad-PCB:WS2812B-2020"
 			(at 0 0 90)
 			(layer "F.Fab")
@@
 		)
 	)
-	(footprint "rp2350-launchpad:WS2812B-2020"
+	(footprint "rp2350b-launchpad-PCB:WS2812B-2020"
 		(layer "F.Cu")
 		(at 149.86 139.446 90)
@@
 			)
 		)
-		(property "Footprint" "rp2350-launchpad:WS2812B-2020"
+		(property "Footprint" "rp2350b-launchpad-PCB:WS2812B-2020"
 			(at 0 0 90)
 			(layer "F.Fab")
@@
 		)
 	)
-	(footprint "rp2350-launchpad:WS2812B-2020"
+	(footprint "rp2350b-launchpad-PCB:WS2812B-2020"
 		(layer "F.Cu")
 		(at 152.4 139.446 90)
@@
 			)
 		)
-		(property "Footprint" "rp2350-launchpad:WS2812B-2020"
+		(property "Footprint" "rp2350b-launchpad-PCB:WS2812B-2020"
 			(at 0 0 90)
 			(layer "F.Fab")
@@
 		)
 	)
-	(footprint "rp2350-launchpad:WS2812B-2020"
+	(footprint "rp2350b-launchpad-PCB:WS2812B-2020"
 		(layer "F.Cu")
 		(at 154.94 139.446 90)
@@
 			)
 		)
-		(property "Footprint" "rp2350-launchpad:WS2812B-2020"
+		(property "Footprint" "rp2350b-launchpad-PCB:WS2812B-2020"
 			(at 0 0 90)
 			(layer "F.Fab")
@@
 		)
 	)
-	(footprint "rp2350-launchpad:WS2812B-2020"
+	(footprint "rp2350b-launchpad-PCB:WS2812B-2020"
 		(layer "F.Cu")
 		(at 157.48 139.446 90)
@@
 			)
 		)
-		(property "Footprint" "rp2350-launchpad:WS2812B-2020"
+		(property "Footprint" "rp2350b-launchpad-PCB:WS2812B-2020"
 			(at 0 0 90)
 			(layer "F.Fab")
@@
 		)
 	)
-	(footprint "rp2350-launchpad:WS2812B-2020"
+	(footprint "rp2350b-launchpad-PCB:WS2812B-2020"
 		(layer "F.Cu")
 		(at 139.7 139.446 90)
@@
 			)
 		)
-		(property "Footprint" "rp2350-launchpad:WS2812B-2020"
+		(property "Footprint" "rp2350b-launchpad-PCB:WS2812B-2020"
 			(at 0 0 90)
 			(layer "F.Fab")
@@
 		)
 	)
-	(footprint "rp2350-launchpad:KMR2-Switch"
+	(footprint "rp2350b-launchpad-PCB:KMR2-Switch"
 		(layer "F.Cu")
 		(at 152.424 131.191 -90)
@@
 			)
 		)
-		(property "Footprint" "rp2350-launchpad:KMR2-Switch"
+		(property "Footprint" "rp2350b-launchpad-PCB:KMR2-Switch"
 			(at 0 0 90)
 			(layer "F.Fab")
@@
 		)
 	)
-	(footprint "rp2350-launchpad:PCM13SMTR"
+	(footprint "rp2350b-launchpad-PCB:PCM13SMTR"
 		(layer "F.Cu")
 		(at 112.649 83.566 -90)
@@
 			)
 		)
-		(property "Footprint" "rp2350-launchpad:PCM13SMTR"
+		(property "Footprint" "rp2350b-launchpad-PCB:PCM13SMTR"
 			(at 0 0 -90)
 			(layer "F.Fab")
@@
 		)
 	)
-	(footprint "rp2350-launchpad:USB-C-GCT-USB4105"
+	(footprint "rp2350b-launchpad-PCB:USB-C-GCT-USB4105"
 		(layer "F.Cu")
 		(at 122.555 145.355)
@@
 			)
 		)
-		(property "Footprint" "rp2350-launchpad:USB-C-GCT-USB4105"
+		(property "Footprint" "rp2350b-launchpad-PCB:USB-C-GCT-USB4105"
 			(at -16.4 -8.67 0)
 			(layer "F.Fab")
@@
 		)
 	)
-	(footprint "rp2350-launchpad:DIPT-1188E"
+	(footprint "rp2350b-launchpad-PCB:DIPT-1188E"
 		(layer "F.Cu")
 		(at 113.126 99.829 -90)
@@
 			)
 		)
-		(property "Footprint" "rp2350-launchpad:DIPT-1188E"
+		(property "Footprint" "rp2350b-launchpad-PCB:DIPT-1188E"
 			(at 0 0 90)
 			(layer "F.Fab")
@@
 		)
 	)
-	(footprint "rp2350-launchpad:DIPT-1188E"
+	(footprint "rp2350b-launchpad-PCB:DIPT-1188E"
 		(layer "F.Cu")
 		(at 166.24 99.88 90)
@@
 			)
 		)
-		(property "Footprint" "rp2350-launchpad:DIPT-1188E"
+		(property "Footprint" "rp2350b-launchpad-PCB:DIPT-1188E"
 			(at 0 0 90)
 			(layer "F.Fab")
@@
 		)
 	)
-	(footprint "rp2350-launchpad:USB-C-GCT-USB4105"
+	(footprint "rp2350b-launchpad-PCB:USB-C-GCT-USB4105"
 		(layer "F.Cu")
 		(at 122.557 73.014 180)
@@
 			)
 		)
-		(property "Footprint" "rp2350-launchpad:USB-C-GCT-USB4105"
+		(property "Footprint" "rp2350b-launchpad-PCB:USB-C-GCT-USB4105"
 			(at -16.4 -8.67 0)
 			(layer "F.Fab")
@@
 		)
 	)
-	(footprint "rp2350-launchpad:JST-S2B-PH-KL"
+	(footprint "rp2350b-launchpad-PCB:JST-S2B-PH-KL"
 		(layer "B.Cu")
 		(at 131.127 84.419 -90)
@@
 			)
 		)
-		(property "Footprint" "rp2350-launchpad:JST-S2B-PH-KL"
+		(property "Footprint" "rp2350b-launchpad-PCB:JST-S2B-PH-KL"
 			(at 0 0 90)
 			(layer "B.Fab")
