File: rp2350b-launchpad-PCB.kicad_sch (KiCad schematic)
At the start: 1 part, among them J1 Target Isolation Jumpers

Commit message: Ready for Version v1.0. Changed PCB to comply with RPi design 'rules'. Without using special components and PCB designs, the PCB may not be produced :\
Other:
- title: RP2040 Launchpad -> RP2350 Launchpad
Changed lines of the file:
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@@
 	(paper "A4")
 	(title_block
-		(title "RP2040 Launchpad")
-		(date "2022-02-06")
-		(rev "v0.1")
+		(title "RP2350 Launchpad")
+		(date "2024-12-10")
+		(rev "v1.0")
 		(company "ISS Intelligent Sensor Solutions")
-		(comment 1 "Created by A. Terstegge")
-		(comment 2 "A TI-style Launchpad with RP2040 MCU")
+		(comment 1 "(C) 2024 A. Terstegge")
+		(comment 2 "and integrated RP2040-based debugger")
+		(comment 3 "A TI-style Launchpad with RP2350 MCU")
 	)
 	(junction
