File: Target.kicad_sch (KiCad schematic)
At the start: 62 parts, among them J10 PWR Header, J11 LP Extension Heder, J12 LP Header right, J13 PWR Header, J8 Jumper, J9 LP Header left, SW2 RESET, SW3 BOOT, U10 WS2812B-2020, U11 WS2812B-2020, U12 WS2812B-2020, U13 WS2812B-2020, U14 WS2812B-2020, U15 WS2812B-2020, U16 WS2812B-2020, U6 25Q64, U7 APS6404L-3SQR, U8 RP2350_80QFN, U9 WS2812B-2020, Y2 12MHz

Commit message: Renumbering parts on target.
Parts:
- renumbered C24 to C23, C25 to C24, C26 to C25, C27 to C26, C28 to C27, C29 to C28, C30 to C29, C31 to C30, C32 to C31, C33 to C32, C34 to C33, C35 to C34, C36 to C35, C37 to C36, C38 to C37, C39 to C38, C40 to C39, C41 to C40
Changed lines of the file:
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@@
 		(on_board yes)
 		(dnp no)
-		(property "Reference" "#PWR045"
+		(property "Reference" "#PWR046"
 			(at 190.5 36.83 0)
 			(effects
@@
 			(project ""
 				(path "/60290668-847e-40fe-8544-1cbbc26023b6/00000000-0000-0000-0000-0000626cc112"
-					(reference "#PWR045")
+					(reference "#PWR046")
 					(unit 1)
 				)
@@
 		(on_board yes)
 		(dnp no)
-		(property "Reference" "#PWR044"
+		(property "Reference" "#PWR045"
 			(at 190.5 26.67 0)
 			(effects
@@
 			(project ""
 				(path "/60290668-847e-40fe-8544-1cbbc26023b6/00000000-0000-0000-0000-0000626cc112"
-					(reference "#PWR044")
+					(reference "#PWR045")
 					(unit 1)
 				)
@@
 		(on_board yes)
 		(dnp no)
-		(property "Reference" "C33"
+		(property "Reference" "C32"
 			(at 131.445 20.955 0)
 			(effects
@@
 			(project ""
 				(path "/60290668-847e-40fe-8544-1cbbc26023b6/00000000-0000-0000-0000-0000626cc112"
-					(reference "C33")
+					(reference "C32")
 					(unit 1)
 				)
@@
 		(on_board yes)
 		(dnp no)
-		(property "Reference" "C34"
+		(property "Reference" "C33"
 			(at 137.795 20.955 0)
 			(effects
@@
 			(project ""
 				(path "/60290668-847e-40fe-8544-1cbbc26023b6/00000000-0000-0000-0000-0000626cc112"
-					(reference "C34")
+					(reference "C33")
 					(unit 1)
 				)
@@
 		(on_board yes)
 		(dnp no)
-		(property "Reference" "C35"
+		(property "Reference" "C34"
 			(at 144.145 20.955 0)
 			(effects
@@
 			(project ""
 				(path "/60290668-847e-40fe-8544-1cbbc26023b6/00000000-0000-0000-0000-0000626cc112"
-					(reference "C35")
+					(reference "C34")
 					(unit 1)
 				)
@@
 		(on_board yes)
 		(dnp no)
-		(property "Reference" "C36"
+		(property "Reference" "C35"
 			(at 150.495 20.955 0)
 			(effects
@@
 			(project ""
 				(path "/60290668-847e-40fe-8544-1cbbc26023b6/00000000-0000-0000-0000-0000626cc112"
-					(reference "C36")
+					(reference "C35")
 					(unit 1)
 				)
@@
 		(on_board yes)
 		(dnp no)
-		(property "Reference" "C37"
+		(property "Reference" "C36"
 			(at 156.845 20.955 0)
 			(effects
@@
 			(project ""
 				(path "/60290668-847e-40fe-8544-1cbbc26023b6/00000000-0000-0000-0000-0000626cc112"
-					(reference "C37")
+					(reference "C36")
 					(unit 1)
 				)
@@
 		(on_board yes)
 		(dnp no)
-		(property "Reference" "C38"
+		(property "Reference" "C37"
 			(at 163.195 20.955 0)
 			(effects
@@
 			(project ""
 				(path "/60290668-847e-40fe-8544-1cbbc26023b6/00000000-0000-0000-0000-0000626cc112"
-					(reference "C38")
+					(reference "C37")
 					(unit 1)
 				)
@@
 		(on_board yes)
 		(dnp no)
-		(property "Reference" "C32"
+		(property "Reference" "C31"
 			(at 125.095 20.955 0)
 			(effects
@@
 			(project ""
 				(path "/60290668-847e-40fe-8544-1cbbc26023b6/00000000-0000-0000-0000-0000626cc112"
-					(reference "C32")
+					(reference "C31")
 					(unit 1)
 				)
@@
 		(on_board yes)
 		(dnp no)
-		(property "Reference" "C28"
+		(property "Reference" "C27"
 			(at 40.64 82.55 90)
 			(effects
@@
 			(project ""
 				(path "/60290668-847e-40fe-8544-1cbbc26023b6/00000000-0000-0000-0000-0000626cc112"
-					(reference "C28")
+					(reference "C27")
 					(unit 1)
 				)
@@
 		(on_board yes)
 		(dnp no)
-		(property "Reference" "C27"
+		(property "Reference" "C26"
 			(at 40.64 72.39 90)
 			(effects
@@
 			(project ""
 				(path "/60290668-847e-40fe-8544-1cbbc26023b6/00000000-0000-0000-0000-0000626cc112"
-					(reference "C27")
+					(reference "C26")
 					(unit 1)
 				)
@@
 		(on_board yes)
 		(dnp no)
-		(property "Reference" "#PWR046"
+		(property "Reference" "#PWR044"
 			(at 186.69 123.19 0)
 			(effects
@@
 			(project "rp2350b-launchpad-PCB"
 				(path "/60290668-847e-40fe-8544-1cbbc26023b6/00000000-0000-0000-0000-0000626cc112"
-					(reference "#PWR046")
+					(reference "#PWR044")
 					(unit 1)
 				)
@@
 		(on_board yes)
 		(dnp no)
-		(property "Reference" "C24"
+		(property "Reference" "C23"
 			(at 38.1 45.72 90)
 			(effects
@@
 			(project "rp2350b-launchpad-PCB"
 				(path "/60290668-847e-40fe-8544-1cbbc26023b6/00000000-0000-0000-0000-0000626cc112"
-					(reference "C24")
+					(reference "C23")
 					(unit 1)
 				)
@@
 		(on_board yes)
 		(dnp no)
-		(property "Reference" "C26"
+		(property "Reference" "C25"
 			(at 38.1 60.96 90)
 			(effects
@@
 			(project "rp2350b-launchpad-PCB"
 				(path "/60290668-847e-40fe-8544-1cbbc26023b6/00000000-0000-0000-0000-0000626cc112"
-					(reference "C26")
+					(reference "C25")
 					(unit 1)
 				)
@@
 		(on_board yes)
 		(dnp no)
-		(property "Reference" "C29"
+		(property "Reference" "C28"
 			(at 53.975 20.955 0)
 			(effects
@@
 			(project "rp2350b-launchpad-PCB"
 				(path "/60290668-847e-40fe-8544-1cbbc26023b6/00000000-0000-0000-0000-0000626cc112"
-					(reference "C29")
+					(reference "C28")
 					(unit 1)
 				)
@@
 		(on_board yes)
 		(dnp no)
-		(property "Reference" "C30"
+		(property "Reference" "C29"
 			(at 61.595 20.955 0)
 			(effects
@@
 			(project "rp2350b-launchpad-PCB"
 				(path "/60290668-847e-40fe-8544-1cbbc26023b6/00000000-0000-0000-0000-0000626cc112"
-					(reference "C30")
+					(reference "C29")
 					(unit 1)
 				)
@@
 		(on_board yes)
 		(dnp no)
-		(property "Reference" "C25"
+		(property "Reference" "C24"
 			(at 34.29 52.705 90)
 			(effects
@@
 			(project "rp2350b-launchpad-PCB"
 				(path "/60290668-847e-40fe-8544-1cbbc26023b6/00000000-0000-0000-0000-0000626cc112"
-					(reference "C25")
+					(reference "C24")
 					(unit 1)
 				)
@@
 		(on_board yes)
 		(dnp no)
-		(property "Reference" "C31"
+		(property "Reference" "C30"
 			(at 69.215 20.955 0)
 			(effects
@@
 			(project "rp2350b-launchpad-PCB"
 				(path "/60290668-847e-40fe-8544-1cbbc26023b6/00000000-0000-0000-0000-0000626cc112"
-					(reference "C31")
+					(reference "C30")
 					(unit 1)
 				)
@@
 		(on_board yes)
 		(dnp no)
-		(property "Reference" "C39"
+		(property "Reference" "C38"
 			(at 169.545 20.955 0)
 			(effects
@@
 			(project "rp2350b-launchpad-PCB"
 				(path "/60290668-847e-40fe-8544-1cbbc26023b6/00000000-0000-0000-0000-0000626cc112"
-					(reference "C39")
+					(reference "C38")
 					(unit 1)
 				)
@@
 		(on_board yes)
 		(dnp no)
-		(property "Reference" "C41"
+		(property "Reference" "C40"
 			(at 182.245 20.955 0)
 			(effects
@@
 			(project "rp2350b-launchpad-PCB"
 				(path "/60290668-847e-40fe-8544-1cbbc26023b6/00000000-0000-0000-0000-0000626cc112"
-					(reference "C41")
+					(reference "C40")
 					(unit 1)
 				)
@@
 		(on_board yes)
 		(dnp no)
-		(property "Reference" "C40"
+		(property "Reference" "C39"
 			(at 175.895 20.955 0)
 			(effects
@@
 			(project "rp2350b-launchpad-PCB"
 				(path "/60290668-847e-40fe-8544-1cbbc26023b6/00000000-0000-0000-0000-0000626cc112"
-					(reference "C40")
+					(reference "C39")
 					(unit 1)
 				)

Commit message: Ready for Version v1.0. Changed PCB to comply with RPi design 'rules'. Without using special components and PCB designs, the PCB may not be produced :\
Parts:
- added J10, J8, J9: Jumper, Jumper:SolderJumper-2_P1.3mm_Bridged_RoundedPad1.0x1.5mm, symbol rp2350b-launchpad-PCB:Jumper
- C25: footprint Capacitor_SMD:C_0402_1005Metric -> Capacitor_SMD:C_0603_1608Metric
- C26, C27: value 22pF -> 15pF
- L2: value 4u7 -> 3u3; footprint Inductor_SMD:L_1008_2520Metric -> rp2350b-launchpad-PCB:AOTA-B201610S3R3-101-T
- USB2: footprint rp2350b-launchpad-PCB:USB-C-GCT-USB4105 -> rp2350b-launchpad-PCB:GT-USB-7010B
- renumbered J8 to J11, J9 to J12, J10 to J13, J11 to J14, J12 to J15, J13 to J16
Connections:
- net at U9.3 (DIN): now also J8.2; no longer U8.48 (GPIO39)
- net at U8.37 (GPIO29): now also J10.1; no longer R32.1
- net at R31.1: now also J9.2; no longer U8.36 (GPIO28)
- new net: J10.2, R32.1
- new net: J8.1, U8.48 (GPIO39)
- new net: J9.1, U8.36 (GPIO28)
Other:
- company: (none) -> ISS Intelligent Sensor Solutions
- title: (none) -> RP2350 Launchpad
- moved on the sheet: C21, C22, D6, J11, R28, R29, R30, R31, R32, R33, S1, S2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

Commit message: Updates for better JLCPCB processing. Version is now 1.1
Parts:
- C21: value 4,7u -> 4u7; Hersteller (none) -> Samsung Electro-Mechanics; JLCPCB Part # (none) -> C23733
- C22, C31, C32, C33, C34, C35, C36, C37, C38, C39, C40: Hersteller (none) -> Samsung Electro-Mechanics; JLCPCB Part # (none) -> C1525
- C23, C25: value 4.7u -> 4u7; Hersteller (none) -> Samsung Electro-Mechanics; JLCPCB Part # (none) -> C19666
- C24, C29: value 4.7u -> 4u7; Hersteller (none) -> Samsung Electro-Mechanics; JLCPCB Part # (none) -> C23733
- C26, C27: Hersteller (none) -> FH (Guangdong Fenghua Advanced Tech); JLCPCB Part # (none) -> C1548; MANUFACTURER z.B. Kemet -> (none); STANDARD unkritisch -> (none)
- C28, C30: value 100n -> 100nF; Hersteller (none) -> Samsung Electro-Mechanics; JLCPCB Part # (none) -> C1525
- D6: Hersteller (none) -> Hubei KENTO Elec; JLCPCB Part # (none) -> C2286
- L2: value 3u3 -> 4u7; Hersteller (none) -> Abracon LLC; JLCPCB Part # (none) -> C42411119
- R17: Hersteller (none) -> UNI-ROYAL(Uniroyal Elec); JLCPCB Part # (none) -> C25803; STANDARD unkritisch -> (none)
- R18: Hersteller (none) -> UNI-ROYAL(Uniroyal Elec); JLCPCB Part # (none) -> C25161
- R19, R20: Hersteller (none) -> UNI-ROYAL(Uniroyal Elec); JLCPCB Part # (none) -> C23186
- R21, R27, R28, R29, R30, R31, R32: Hersteller (none) -> UNI-ROYAL(Uniroyal Elec); JLCPCB Part # (none) -> C11702
- R22, R23: Hersteller (none) -> YAGEO; JLCPCB Part # (none) -> C137890; STANDARD unkritisch -> (none)
- R24, R25: Hersteller (none) -> UNI-ROYAL(Uniroyal Elec); JLCPCB Part # (none) -> C25531; STANDARD unkritisch -> (none)
- R26: Hersteller (none) -> UNI-ROYAL(Uniroyal Elec); JLCPCB Part # (none) -> C25804
- R33: Hersteller (none) -> UNI-ROYAL(Uniroyal Elec); JLCPCB Part # (none) -> C23179
- S1, S2, SW2: Hersteller (none) -> Diptronics; JLCPCB Part # (none) -> C240289
- SW3: Hersteller (none) -> C&K; JLCPCB Part # (none) -> C221680
- U10, U11, U12, U13, U14, U15, U16, U9: Hersteller (none) -> Worldsemi; JLCPCB Part # (none) -> C965555
- U6: Hersteller (none) -> Winbond Elec; JLCPCB Part # (none) -> C2940197
- U7: Hersteller (none) -> AP Memory; JLCPCB Part # (none) -> C3040877
- U8: Hersteller (none) -> Raspberry Pi; JLCPCB Part # (none) -> C42415655
- USB2: value USB-C-Socket -> USB-C Connector; Hersteller (none) -> G-Switch; JLCPCB Part # (none) -> C2837092
- Y2: footprint Crystal:Crystal_SMD_TXC_7M-4Pin_3.2x2.5mm -> Crystal:Crystal_SMD_Abracon_ABM8AIG-4Pin_3.2x2.5mm; Hersteller (none) -> Abracon LLC; JLCPCB Part # (none) -> C20625731

Commit message: Ready for v1.1
Connections:
- net I2C0_SCL: now also U8.7 (GPIO9); no longer U8.78 (GPIO1)
- net I2C0_SDA: now also U8.6 (GPIO8); no longer U8.77 (GPIO0)
- net ~{RAM_CS}: now also U8.77 (GPIO0); no longer U8.79 (GPIO2)
- net GPIO8 renamed GPIO1
- net GPIO1: now also U8.78 (GPIO1); no longer U8.6 (GPIO8)
- net GPIO9 renamed GPIO2
- net GPIO2: now also U8.79 (GPIO2); no longer U8.7 (GPIO9)
Changed lines of the file:
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@@
 		)
 	)
-	(label "GPIO8"
+	(label "GPIO1"
 		(at 270.51 60.96 180)
 		(effects
@@
 		)
 	)
-	(label "GPIO8"
-		(at 149.86 60.96 180)
+	(label "GPIO2"
+		(at 149.86 45.72 180)
 		(effects
 			(font
@@
 	)
 	(label "I2C0_SCL"
-		(at 149.86 43.18 180)
+		(at 149.86 63.5 180)
 		(effects
 			(font
@@
 		)
 	)
-	(label "GPIO9"
+	(label "GPIO2"
 		(at 241.3 60.96 0)
 		(effects
@@
 		)
 	)
-	(label "GPIO9"
-		(at 149.86 63.5 180)
+	(label "GPIO1"
+		(at 149.86 43.18 180)
 		(effects
 			(font
@@
 	)
 	(label "I2C0_SDA"
-		(at 149.86 40.64 180)
+		(at 149.86 60.96 180)
 		(effects
 			(font
@@
 	)
 	(label "~{RAM_CS}"
-		(at 149.86 45.72 180)
-		(effects
-			(font
+		(at 149.86 40.64 180)
+		(effects
+			(font
